File: Common-Miner-Baseboard.kicad_pcb (KiCad board)
At the start: 2 copper layers, 108 x 38 mm, 47 parts, among them J1 EXP1, J10 EXP10, J11 EXP11, J12 EXP, J2 EXP2, J3 EXP3, J4 EXP4, J5 EXP5, J6 EXP6, J7 EXP7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

Commit message: Updated project for KiCad 7 & added Gerber Files
Other:
- net class Default removed
